File: schematics/CortexBoard 40x/CortexBoard.kicad_pcb (KiCad board)
At the start: 2 copper layers, 37 parts, among them J1 LEG1-LO, J10 LEG2-LO, J12 LEG2-HI, J13 LEG3-LO, J14 LEG3-HI, J15 LEG4-LO, J16 LEG4-HI, J17 LEG5-LO, J18 LEG5-HI, J2 UART6 Connector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

Commit message: no message
Parts:
- moved D2 6.98 mm to (196.8, 73.0)
- moved J3 6.98 mm to (215.9, 108.6)
- moved J4 6.98 mm to (177.8, 103.5)
- moved J5 6.98 mm to (196.8, 127.6)
- moved J9 6.98 mm to (215.9, 103.5)
- moved P1 6.98 mm to (177.8, 108.6)
- moved P10 6.98 mm to (175.3, 83.2)
- moved P3 6.98 mm to (204.5, 103.5)
- moved Q1 6.98 mm to (185.4, 73.0)
- moved R4 6.98 mm to (213.4, 121.3)
- moved R5 6.98 mm to (231.1, 98.4)
- moved REL1 6.98 mm to (200.7, 73.0)
- moved P6 1.27 mm to (120.7, 138.4)
- moved SW2 0.63 mm to (114.9, 138.4)
Routing:
- net Net-(P6-Pad1): track 0.00 -> 5.72 mm
- net /GND: track 413.7 -> 411.6 mm

Commit message: no message
Parts:
- moved J1 2.54 mm to (141.0, 109.2)
- moved J17 2.54 mm to (141.0, 94.0)
Routing:
- net /+14V: track 365.5 -> 350.2 mm
- net /+10V: track 246.7 -> 236.6 mm
- net /RX2: track 143.5 -> 148.6 mm
- net /GND: track 411.6 -> 407.2 mm
- net /TX2: track 154.5 -> 152.0 mm
